File: pchMosFet_mod.kicad_pcb (KiCad board)
At the start: 2 copper layers, 14 x 44 mm, 8 parts, among them J1 LOAD, J2 Conn_01x03_Pin, Q1 2SC1815, Q2 PMOS

Commit message: VCC/GNDラインの電流容量修正
Parts:
- moved Q2 1.27 mm to (96.5, 67.6)
Routing:
- net GND: track 50.0 -> 12.3 mm, vias 1 -> 0
- net Net-(Q1-C): track 20.1 -> 24.8 mm
- net Net-(Q2-G): track 14.6 -> 9.98 mm
- net VCC: track 31.5 -> 28.2 mm
- net Net-(Q1-B): track 15.0 -> 18.1 mm
- net Net-(J1-Pin_2): track 17.2 -> 15.4 mm
- net TRIG: track 21.2 -> 20.4 mm, vias 2 -> 1
Other:
- board text added: "Ver.2"
